Commit message: ...

File: description/robot_core.xacro (robot description, xacro)
@@ -73,8 +73,8 @@
   </visual>
   <collision>
-    <!-- <origin xyz="0.071 -0.121 -0.0325" rpy="0 0 0"/> -->
+    <origin xyz="0.071 -0.121 -0.0325" rpy="0 0 0"/>
     <geometry>
-      <!-- <mesh filename="file://$(find bot)/meshes/LR_wheel.stl" scale="0.001 0.001 0.001"/> -->
-      <sphere radius="0.0325"/>
+      <mesh filename="file://$(find bot)/meshes/LR_wheel.stl" scale="0.001 0.001 0.001"/>
+      <!-- <sphere radius="0.0325"/> -->
     </geometry>
   </collision>
@@ -175,8 +175,8 @@
   </visual>
   <collision>
-    <!-- <origin xyz="0.071 0.121 -0.0325" rpy="0 0 0"/> -->
+    <origin xyz="0.071 0.121 -0.0325" rpy="0 0 0"/>
     <geometry>
-      <!-- <mesh filename="file://$(find bot)/meshes/RR_wheel.stl" scale="0.001 0.001 0.001"/> -->
-      <sphere radius="0.0325"/>
+      <mesh filename="file://$(find bot)/meshes/RR_wheel.stl" scale="0.001 0.001 0.001"/>
+      <!-- <sphere radius="0.0325"/> -->
     </geometry>
   </collision>
